Commit message: rviz vizes

File: src/interfaces/udrf/sjtu_drone.urdf (robot description, URDF)
Before this commit: robot sjtu_drone, 5 links, 4 joints
Links:
- link base_link: geometry collision mesh filename=package://interfaces/udrf/quadrotor_4.stl; visual mesh filename=package://interfaces/udrf/quadrotor_4.dae
